File: KiCad files/Env-F12TKL.kicad_sch (KiCad schematic)
At the start: 214 parts, among them J1 TSA343G00-250J2, U1 SOT-23-5 5.5V 3.3V 500mA, U2 RP2040

Commit message: a lot of general re-work
Parts:
- removed D_5: 1N4148W, Diode_SMD:D_SOD-123, symbol Device:D_Small
- removed K_5: KEYSW, EnvExtras:MXOnly-1U-Hotswap-Modified, symbol MX_Alps_Hybrid:MX-NoLED
- added D_52: 1N4148W, Diode_SMD:D_SOD-123, symbol Device:D_Small
- added K_91: KEYSW, EnvExtras:MXOnly-1U-Hotswap-Modified, symbol MX_Alps_Hybrid:MX-NoLED
- Stab1: footprint Mounting_Keyboard_Stabilizer:Stabilizer_Cherry_MX_7u -> Mounting_Keyboard_Stabilizer:Stabilizer_Cherry_MX_6.25u
Connections:
- net col10: now also K_91.1 (COL)
- net row5: now also D_52.1 (K)
- new net: D_52.2 (A), K_91.2 (ROW)
Changed lines of the file:
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@@
   (junction (at 74.93 57.15) (diameter 0) (color 0 0 0 0)
   )
+  (junction (at 292.1 170.18) (diameter 0) (color 0 0 0 0)
+  )
   (junction (at 430.53 57.15) (diameter 0) (color 0 0 0 0)
   )
@@
   (junction (at 269.24 264.16) (diameter 0) (color 0 0 0 0)
   )
-  (junction (at 201.93 31.75) (diameter 0) (color 0 0 0 0)
-  )
   (junction (at 344.17 260.35) (diameter 0) (color 0 0 0 0)
   )
@@
   (junction (at 455.93 133.35) (diameter 0) (color 0 0 0 0)
   )
-  (junction (at 190.5 43.18) (diameter 0) (color 0 0 0 0)
-  )
   (junction (at 232.41 269.24) (diameter 0) (color 0 0 0 0)
   )
@@
   (junction (at 215.9 119.38) (diameter 0) (color 0 0 0 0)
   )
+  (junction (at 303.53 133.35) (diameter 0) (color 0 0 0 0)
+  )
   (junction (at 227.33 107.95) (diameter 0) (color 0 0 0 0)
   )
@@
     (stroke (width 0) (type default) (color 0 0 0 0))
   )
-  (wire (pts (xy 201.93 31.75) (xy 201.93 57.15))
+  (wire (pts (xy 201.93 24.13) (xy 201.93 57.15))
     (stroke (width 0) (type default) (color 0 0 0 0))
   )
@@
     (stroke (width 0) (type default) (color 0 0 0 0))
   )
-  (wire (pts (xy 303.53 133.35) (xy 303.53 107.95))
+  (wire (pts (xy 303.53 107.95) (xy 303.53 133.35))
     (stroke (width 0) (type default) (color 0 0 0 0))
   )
@@
     (stroke (width 0) (type default) (color 0 0 0 0))
   )
-  (wire (pts (xy 215.9 170.18) (xy 317.5 170.18))
+  (wire (pts (xy 215.9 170.18) (xy 292.1 170.18))
     (stroke (width 0) (type default) (color 0 0 0 0))
   )
@@
     (stroke (width 0) (type default) (color 0 0 0 0))
   )
-  (wire (pts (xy 139.7 43.18) (xy 190.5 43.18))
+  (wire (pts (xy 139.7 43.18) (xy 215.9 43.18))
     (stroke (width 0) (type default) (color 0 0 0 0))
   )
@@
     (stroke (width 0) (type default) (color 0 0 0 0))
   )
+  (wire (pts (xy 303.53 133.35) (xy 303.53 158.75))
+    (stroke (width 0) (type default) (color 0 0 0 0))
+  )
   (wire (pts (xy 342.9 87.63) (xy 342.9 88.9))
     (stroke (width 0) (type default) (color 0 0 0 0))
@@
     (stroke (width 0) (type default) (color 0 0 0 0))
   )
-  (wire (pts (xy 195.58 31.75) (xy 201.93 31.75))
-    (stroke (width 0) (type default) (color 0 0 0 0))
-  )
   (wire (pts (xy 269.24 264.16) (xy 269.24 269.24))
     (stroke (width 0) (type default) (color 0 0 0 0))
@@
     (stroke (width 0) (type default) (color 0 0 0 0))
   )
+  (wire (pts (xy 292.1 170.18) (xy 317.5 170.18))
+    (stroke (width 0) (type default) (color 0 0 0 0))
+  )
   (wire (pts (xy 449.58 82.55) (xy 455.93 82.55))
     (stroke (width 0) (type default) (color 0 0 0 0))
@@
     (stroke (width 0) (type default) (color 0 0 0 0))
   )
-  (wire (pts (xy 201.93 24.13) (xy 201.93 31.75))
-    (stroke (width 0) (type default) (color 0 0 0 0))
-  )
   (wire (pts (xy 256.54 269.24) (xy 259.08 269.24))
     (stroke (width 0) (type default) (color 0 0 0 0))
@@
     (stroke (width 0) (type default) (color 0 0 0 0))
   )
-  (wire (pts (xy 190.5 36.83) (xy 190.5 38.1))
-    (stroke (width 0) (type default) (color 0 0 0 0))
-  )
   (wire (pts (xy 284.48 358.14) (xy 299.72 358.14))
     (stroke (width 0) (type default) (color 0 0 0 0))
@@
     (stroke (width 0) (type default) (color 0 0 0 0))
   )
-  (wire (pts (xy 190.5 43.18) (xy 215.9 43.18))
-    (stroke (width 0) (type default) (color 0 0 0 0))
-  )
   (wire (pts (xy 322.58 257.81) (xy 322.58 260.35))
     (stroke (width 0) (type default) (color 0 0 0 0))
@@
     (stroke (width 0) (type default) (color 0 0 0 0))
   )
+  (wire (pts (xy 297.18 158.75) (xy 303.53 158.75))
+    (stroke (width 0) (type default) (color 0 0 0 0))
+  )
   (wire (pts (xy 38.1 43.18) (xy 63.5 43.18))
     (stroke (width 0) (type default) (color 0 0 0 0))
   )
+  (wire (pts (xy 292.1 163.83) (xy 292.1 165.1))
+    (stroke (width 0) (type default) (color 0 0 0 0))
+  )
   (wire (pts (xy 284.48 299.72) (xy 299.72 299.72))
     (stroke (width 0) (type default) (color 0 0 0 0))
@@
       (effects (font (size 1.27 1.27)) (justify left))
     )
-    (property "Footprint" "Mounting_Keyboard_Stabilizer:Stabilizer_Cherry_MX_7u" (id 2) (at 140.97 204.47 0)
+    (property "Footprint" "Mounting_Keyboard_Stabilizer:Stabilizer_Cherry_MX_6.25u" (id 2) (at 140.97 204.47 0)
       (effects (font (size 1.27 1.27)) hide)
     )
@@
     (pin "2")
   )
-  (symbol (lib_id "MX_Alps_Hybrid:MX-NoLED") (at 191.77 33.02 0) (unit 1)
-    (in_bom yes) (on_board yes)
-    (property "Reference" "K_5" (id 0) (at 191.77 27.1018 0)
-      (effects (font (size 1.524 1.524)))
-    )
-    (property "Value" "KEYSW" (id 1) (at 191.77 35.56 0)
-      (effects (font (size 1.524 1.524)) hide)
-    )
-    (property "Footprint" "EnvExtras:MXOnly-1U-Hotswap-Modified" (id 2) (at 191.77 33.02 0)
-      (effects (font (size 1.524 1.524)) hide)
-    )
-    (property "Datasheet" "" (id 3) (at 191.77 33.02 0)
-      (effects (font (size 1.524 1.524)))
-    )
-    (pin "1")
-    (pin "2")
-  )
   (symbol (lib_id "Regulator_Linear:AP131-15") (at 93.98 259.08 0) (unit 1)
     (in_bom yes) (on_board yes)
@@
     (pin "2")
   )
-  (symbol (lib_id "Device:D_Small") (at 190.5 40.64 90) (unit 1)
-    (in_bom yes) (on_board yes)
-    (property "Reference" "D_5" (id 0) (at 193.04 38.862 90)
-      (effects (font (size 1.27 1.27)) (justify right))
-    )
-    (property "Value" "1N4148W" (id 1) (at 193.04 41.148 90)
-      (effects (font (size 1.27 1.27)) (justify right))
-    )
-    (property "Footprint" "Diode_SMD:D_SOD-123" (id 2) (at 191.77 48.26 0)
-      (effects (font (size 1.27 1.27)) hide)
-    )
-    (property "Datasheet" "~" (id 3) (at 191.77 48.26 0)
-      (effects (font (size 1.27 1.27)) hide)
-    )
-    (pin "1")
-    (pin "2")
-  )
   (symbol (lib_id "Device:D_Small") (at 266.7 91.44 90) (unit 1)
     (in_bom yes) (on_board yes)
@@
     (pin "2")
   )
+  (symbol (lib_id "MX_Alps_Hybrid:MX-NoLED") (at 293.37 160.02 0) (unit 1)
+    (in_bom yes) (on_board yes)
+    (property "Reference" "K_91" (id 0) (at 293.37 154.1018 0)
+      (effects (font (size 1.524 1.524)))
+    )
+    (property "Value" "KEYSW" (id 1) (at 293.37 162.56 0)
+      (effects (font (size 1.524 1.524)) hide)
+    )
+    (property "Footprint" "EnvExtras:MXOnly-1U-Hotswap-Modified" (id 2) (at 293.37 160.02 0)
+      (effects (font (size 1.524 1.524)) hide)
+    )
+    (property "Datasheet" "" (id 3) (at 293.37 160.02 0)
+      (effects (font (size 1.524 1.524)))
+    )
+    (pin "1")
+    (pin "2")
+  )
   (symbol (lib_id "MX_Alps_Hybrid:MX-NoLED") (at 217.17 33.02 0) (unit 1)
     (in_bom yes) (on_board yes)
@@
     (pin "2")
   )
+  (symbol (lib_id "Device:D_Small") (at 292.1 167.64 90) (unit 1)
+    (in_bom yes) (on_board yes)
+    (property "Reference" "D_52" (id 0) (at 294.64 165.862 90)
+      (effects (font (size 1.27 1.27)) (justify right))
+    )
+    (property "Value" "1N4148W" (id 1) (at 294.64 168.148 90)
+      (effects (font (size 1.27 1.27)) (justify right))
+    )
+    (property "Footprint" "Diode_SMD:D_SOD-123" (id 2) (at 293.37 175.26 0)
+      (effects (font (size 1.27 1.27)) hide)
+    )
+    (property "Datasheet" "~" (id 3) (at 293.37 175.26 0)
+      (effects (font (size 1.27 1.27)) hide)
+    )
+    (pin "1")
+    (pin "2")
+  )
   (symbol (lib_id "MX_Alps_Hybrid:MX-NoLED") (at 267.97 109.22 0) (unit 1)
     (in_bom yes) (on_board yes)
@@
       (reference "D_4") (unit 1) (value "1N4148W") (footprint "Diode_SMD:D_SOD-123")
     )
-    (path "/b5be3aee-a3aa-4bf1-8c8a-c2f862e4eb93"
-      (reference "D_5") (unit 1) (value "1N4148W") (footprint "Diode_SMD:D_SOD-123")
-    )
     (path "/32e185dc-1352-4d40-ac72-3c6395559690"
       (reference "D_6") (unit 1) (value "1N4148W") (footprint "Diode_SMD:D_SOD-123")
@@
       (reference "D_51") (unit 1) (value "1N4148W") (footprint "Diode_SMD:D_SOD-123")
     )
+    (path "/c555786c-7744-411b-b4bd-34475b8fe87b"
+      (reference "D_52") (unit 1) (value "1N4148W") (footprint "Diode_SMD:D_SOD-123")
+    )
     (path "/929b0dec-b90a-49f3-96a0-1e6f1a29a2ed"
       (reference "D_53") (unit 1) (value "1N4148W") (footprint "Diode_SMD:D_SOD-123")
@@
       (reference "K_4") (unit 1) (value "KEYSW") (footprint "EnvExtras:MXOnly-1U-Hotswap-Modified")
     )
-    (path "/8b852220-4f59-4a64-80a1-bbf574c584b7"
-      (reference "K_5") (unit 1) (value "KEYSW") (footprint "EnvExtras:MXOnly-1U-Hotswap-Modified")
-    )
     (path "/bee2c80e-2a5f-4bc6-ae4a-1789473d2fdf"
       (reference "K_6") (unit 1) (value "KEYSW") (footprint "EnvExtras:MXOnly-1U-Hotswap-Modified")
@@
       (reference "K_90") (unit 1) (value "KEYSW") (footprint "EnvExtras:MXOnly-1U-Hotswap-Modified")
     )
+    (path "/be5985d6-7818-4dbf-93ab-1240698c4324"
+      (reference "K_91") (unit 1) (value "KEYSW") (footprint "EnvExtras:MXOnly-1U-Hotswap-Modified")
+    )
     (path "/39dcd05e-7319-40e9-ae6d-e640fb807318"
       (reference "R4") (unit 1) (value "100K 0402") (footprint "Resistor_SMD:R_0402_1005Metric")
@@
     )
     (path "/6cbe4855-d1e7-4d59-9b56-3b92de6390ab"
-      (reference "Stab1") (unit 1) (value "Stabiliser") (footprint "Mounting_Keyboard_Stabilizer:Stabilizer_Cherry_MX_7u")
+      (reference "Stab1") (unit 1) (value "Stabiliser") (footprint "Mounting_Keyboard_Stabilizer:Stabilizer_Cherry_MX_6.25u")
     )
     (path "/d131b901-3b22-4e81-bde1-64cdb541933a"

Commit message: lots of progress toward wiring up MCU and also added missing crystal
Parts:
- added C15, C16: 22pf 0402, Capacitor_SMD:C_0402_1005Metric, symbol Device:C
- added D_5, D_89: 1N4148W, Diode_SMD:D_SOD-123, symbol Device:D_Small
- added K_5, K_92: KEYSW, EnvExtras:MXOnly-1U-Hotswap-Modified, symbol MX_Alps_Hybrid:MX-NoLED
- added R1: 1K 0402, Resistor_SMD:R_0402_1005Metric, symbol Device:R
- added Stab5: Stabiliser, Mounting_Keyboard_Stabilizer:Stabilizer_Cherry_MX_2u, symbol Mechanical:MountingHole
- added Y1: 3225_4P, Crystal:Crystal_SMD_3225-4Pin_3.2x2.5mm, symbol Device:Crystal_GND24
- Stab1: footprint Mounting_Keyboard_Stabilizer:Stabilizer_Cherry_MX_6.25u -> Mounting_Keyboard_Stabilizer:Stabilizer_Cherry_MX_2u
Connections:
- net GPIO0 is gone; now on net col17: U2.2 (GPIO0)
- net GPIO1 is gone; now on net col16: U2.3 (GPIO1)
- net GPIO10 is gone; now on net col7: U2.13 (GPIO10)
- net GPIO11 is gone; now on net col6: U2.14 (GPIO11)
- net GPIO12 is gone; now on net col5: U2.15 (GPIO12)
- net GPIO13 is gone; now on net col4: U2.16 (GPIO13)
- net GPIO14 is gone; now on net col3: U2.17 (GPIO14)
- net GPIO15 is gone; now on net col2: U2.18 (GPIO15)
- net GPIO16 is gone; now on net col1: U2.27 (GPIO16)
- net GPIO17 is gone; now on net col0: U2.28 (GPIO17)
- net GPIO2 is gone; now on net col15: U2.4 (GPIO2)
- net GPIO3 is gone; now on net col14: U2.5 (GPIO3)
- net GPIO4 is gone; now on net col13: U2.6 (GPIO4)
- net GPIO5 is gone; now on net col12: U2.7 (GPIO5)
- net GPIO6 is gone; now on net col11: U2.8 (GPIO6)
- net GPIO7 is gone; now on net col10: U2.9 (GPIO7)
- net GPIO8 is gone; now on net col9: U2.11 (GPIO8)
- net GPIO9 is gone; now on net col8: U2.12 (GPIO9)
- net GND: now also C15.1, C16.1, Y1.2, Y1.4
- net XIN: now also C15.2, Y1.1
- net XOUT: now also R1.1
- net col1: now also K_80.1 (COL); no longer K_1.1 (COL)
- net col10: now also K_10.1 (COL); no longer K_9.1 (COL)
- net col11: now also K_11.1 (COL); no longer K_10.1 (COL)
- net col12: now also K_12.1 (COL); no longer K_11.1 (COL)
- net col13: now also K_13.1 (COL); no longer K_12.1 (COL)
- net col14: no longer K_13.1 (COL)
- net col2: now also K_1.1 (COL), K_81.1 (COL); no longer K_2.1 (COL), K_80.1 (COL)
- net col3: now also K_2.1 (COL); no longer K_3.1 (COL), K_81.1 (COL)
- net col4: now also K_3.1 (COL), K_5.1 (COL); no longer K_4.1 (COL)
- net col5: now also K_4.1 (COL)
- net col6: now also K_6.1 (COL), K_82.1 (COL)
- net col7: now also K_7.1 (COL); no longer K_6.1 (COL), K_82.1 (COL)
- net col8: now also K_8.1 (COL), K_92.1 (COL); no longer K_7.1 (COL)
- net col9: now also K_9.1 (COL); no longer K_8.1 (COL)
- net row5: now also D_5.1 (K), D_89.1 (K)
- new net: D_5.2 (A), K_5.2 (ROW)
- new net: C16.2, R1.2, Y1.3
- new net: D_89.2 (A), K_92.2 (ROW)
Other:
- note added: "1K resistor to prevent overdriving of the crystal as per the minimal design example"
- note added: "Crystal"
- note added: "RP2040 supports 1MHz to 15MHz"
- note added: "not 22pf but pick to match crystal."
- moved on the sheet: D_1, D_10, D_11, D_12, D_13, D_2, D_3, D_4, D_6, D_7, D_8, D_80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
